File: sem1/aplikacje-mobilne-projekt/pcb/pcb.kicad_pcb (KiCad board)
At the start: 2 copper layers, 18 parts, among them Q1 IRL6283M, Q10 IRL6283M, Q11 IRL6283M, Q12 IRL6283M, Q13 IRL6283M, Q2 IRL6283M, Q3 IRL6283M, Q4 IRL6283M, Q5 IRL6283M, Q6 IRL6283M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

Commit message: pcb design update
Parts:
- added J1: Conn_01x20_Female, Connector_PinHeader_2.54mm:PinHeader_1x20_P2.54mm_Vertical, F.Cu at (79.3, 115.1)
- added J2: Conn_01x20_Female, Connector_PinHeader_2.54mm:PinHeader_1x20_P2.54mm_Vertical, F.Cu at (66.0, 115.0)
- added J3: Conn_01x10_Male, Connector_PinHeader_2.54mm:PinHeader_1x10_P2.54mm_Vertical, F.Cu at (119.9, 120.0)
- added R1: 10k, Resistor_THT:R_Axial_DIN0204_L3.6mm_D1.6mm_P7.62mm_Horizontal, F.Cu at (155.2, 62.0)
- added R2: 10k, Resistor_THT:R_Axial_DIN0204_L3.6mm_D1.6mm_P7.62mm_Horizontal, F.Cu at (93.2, 62.2)
- added R3: 10k, Resistor_THT:R_Axial_DIN0204_L3.6mm_D1.6mm_P7.62mm_Horizontal, F.Cu at (112.2, 62.4)
- added R4: 10k, Resistor_THT:R_Axial_DIN0204_L3.6mm_D1.6mm_P7.62mm_Horizontal, F.Cu at (128.4, 62.2)
- added R5: 10k, Resistor_THT:R_Axial_DIN0204_L3.6mm_D1.6mm_P7.62mm_Horizontal, F.Cu at (144.0, 62.2)
- Q1, Q10, Q11, Q12, Q13, Q2, Q3, Q4, Q5, Q6, Q7, Q8, Q9: value IRL6283M -> IRF540N; footprint Package_DirectFET:DirectFET_MD -> Package_TO_SOT_THT:TO-220-3_Vertical
- U1, U2, U3, U4: value IRF9630PBF -> IRF9540N; footprint footprints:TO220AB_VIS -> Package_TO_SOT_THT:TO-220-3_Vertical
- moved Q5 61.8 mm to (97.0, 100.0), turned to -90 degrees
- moved Q1 51.1 mm to (95.5, 76.9)
- moved D1 42.2 mm to (168.0, 79.1), turned to 90 degrees
- moved Q3 38.8 mm to (125.9, 77.0)
- moved Q2 34.4 mm to (109.5, 76.9)
- moved Q10 34.0 mm to (172.0, 88.0)
- moved Q11 25.4 mm to (156.5, 99.9)
- moved U1 25.3 mm to (97.0, 85.0), turned to -90 degrees
- moved Q13 23.1 mm to (150.5, 113.9)
- moved Q12 21.8 mm to (171.5, 99.9)
- moved Q6 21.1 mm to (111.0, 101.0), turned to -90 degrees
- moved U3 20.5 mm to (127.0, 85.0), turned to -90 degrees
- moved Q7 20.2 mm to (127.0, 101.0), turned to -90 degrees
- moved Q8 18.5 mm to (143.0, 101.0), turned to -90 degrees
- moved Q9 17.6 mm to (156.5, 87.9)
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Connections:
- Q1 pad 1: Net-(R2-Pad2) -> LEFT1
- Q1 pad 2: LEFT1 -> Net-(Q1-Pad2)
- Q10 pad 1: Net-(Q10-Pad1) -> LEFT1
- Q10 pad 2: RIGHT2 -> EMERGENCY
- Q10 pad 3: Gnd -> Net-(Q10-Pad3)
- Q11 pad 1: EMERGENCY -> RIGHT2
- Q11 pad 2: LEFT1 -> Net-(Q11-Pad2)
- Q11 pad 3: Net-(Q11-Pad3) -> Gnd
- Q12 pad 1: Net-(Q11-Pad3) -> LEFT2
- Q12 pad 2: LEFT2 -> Net-(Q10-Pad3)
- Q13 pad 1: Net-(Q13-Pad1) -> EMERGENCY
- Q13 pad 2: EMERGENCY -> Net-(Q13-Pad2)
- Q2 pad 1: Net-(U2-Pad1) -> LEFT2
- Q2 pad 2: LEFT2 -> Net-(Q2-Pad2)
- Q3 pad 1: Net-(M_1-Pad1) -> RIGHT1
- Q3 pad 2: LEFT2 -> Net-(Q3-Pad2)
- Q3 pad 3: Net-(Q13-Pad1) -> Gnd
- Q4 pad 1: Net-(M_1-Pad2) -> RIGHT2
- Q4 pad 2: LEFT1 -> Net-(Q4-Pad2)
- Q4 pad 3: Net-(Q13-Pad1) -> Gnd
- Q5 pad 1: Net-(R4-Pad2) -> LEFT2
- Q5 pad 2: RIGHT1 -> M1
- Q5 pad 3: Gnd -> Net-(Q13-Pad2)
- Q6 pad 1: Net-(R5-Pad2) -> LEFT1
- Q6 pad 2: RIGHT2 -> M2
- Q6 pad 3: Gnd -> Net-(Q13-Pad2)
- Q7 pad 1: Net-(M_2-Pad1) -> RIGHT2
- Q7 pad 2: RIGHT2 -> M3
- Q7 pad 3: Net-(Q13-Pad1) -> Net-(Q13-Pad2)
- Q8 pad 1: Net-(M_2-Pad2) -> RIGHT1
- Q8 pad 2: RIGHT1 -> M4
- Q8 pad 3: Net-(Q13-Pad1) -> Net-(Q13-Pad2)
- Q9 pad 1: EMERGENCY -> RIGHT1
- Q9 pad 2: RIGHT1 -> EMERGENCY
- Q9 pad 3: Net-(Q10-Pad1) -> Net-(Q11-Pad2)
- U1 pad 1: Net-(R2-Pad2) -> Net-(Q1-Pad2)
- U1 pad 2: (no net) -> Vcc
- U1 pad 3: (no net) -> M1
- U2 pad 1: Net-(U2-Pad1) -> Net-(Q2-Pad2)
- U2 pad 2: (no net) -> Vcc
- U2 pad 3: (no net) -> M2
- U3 pad 1: Net-(R4-Pad2) -> Net-(Q3-Pad2)
- U3 pad 2: (no net) -> Vcc
- U3 pad 3: (no net) -> M3
- U4 pad 1: Net-(R5-Pad2) -> Net-(Q4-Pad2)
- U4 pad 2: (no net) -> Vcc
- U4 pad 3: (no net) -> M4
Routing:
- net Vcc: track 0.00 -> 251.8 mm
- net EMERGENCY: track 0.00 -> 29.0 mm
- net Net-(Q1-Pad2): track 0.00 -> 19.1 mm
- net Net-(Q3-Pad2): track 0.00 -> 15.8 mm
- net Net-(Q4-Pad2): track 0.00 -> 15.6 mm
- net Net-(Q2-Pad2): track 0.00 -> 15.5 mm
- net Net-(D1-Pad2): track 0.00 -> 9.07 mm

Commit message: this pcb one actually works
Parts:
- moved Q5 17.7 mm to (87.5, 114.9), turned to 0 degrees
- moved Q8 17.5 mm to (132.5, 114.9), turned to 0 degrees
- moved Q7 16.9 mm to (117.5, 114.9), turned to 0 degrees
- moved Q6 16.4 mm to (102.5, 114.9), turned to 0 degrees
- moved R2 14.3 mm to (97.0, 76.0)
- moved R5 13.8 mm to (144.0, 76.0)
- moved R4 13.8 mm to (128.2, 76.0)
- moved Q1 13.8 mm to (94.5, 90.7)
- moved U4 13.8 mm to (144.0, 98.8)
- moved Q3 13.8 mm to (125.5, 90.8)
- moved Q2 13.8 mm to (109.5, 90.7)
- moved Q4 13.8 mm to (141.5, 90.7)
- moved U1 13.8 mm to (97.0, 98.8)
- moved R3 13.6 mm to (112.0, 76.0)
- moved U2 13.5 mm to (112.0, 98.5)
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Connections:
- J1 pad 14: RIGHT1 -> LEFT1
- J1 pad 15: RIGHT2 -> LEFT2
- J1 pad 16: LEFT1 -> RIGHT1
- J1 pad 17: LEFT2 -> RIGHT2
- U1 pad 2: Vcc -> M1
- U1 pad 3: M1 -> Vcc
- U2 pad 2: Vcc -> M2
- U2 pad 3: M2 -> Vcc
- U3 pad 2: Vcc -> M3
- U3 pad 3: M3 -> Vcc
- U4 pad 2: Vcc -> M4
- U4 pad 3: M4 -> Vcc
Routing:
- net RIGHT1: track 0.00 -> 169.1 mm
- net Net-(Q13-Pad2): track 0.00 -> 124.5 mm
- net M1: track 0.00 -> 114.3 mm
- net M2: track 0.00 -> 86.9 mm
- net M3: track 0.00 -> 75.0 mm
- net RIGHT2: track 0.00 -> 74.5 mm
- net M4: track 0.00 -> 42.7 mm
- net EMERGENCY: track 29.0 -> 66.4 mm
- net LEFT2: track 0.00 -> 34.8 mm
- net LEFT1: track 0.00 -> 18.8 mm
- net Vcc: track 251.8 -> 267.1 mm
- net Net-(Q11-Pad2): track 0.00 -> 13.1 mm
- net Net-(Q10-Pad3): track 0.00 -> 12.3 mm
- net Net-(Q1-Pad2): track 19.1 -> 15.2 mm
- net Net-(D1-Pad2): track 9.07 -> 8.47 mm
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
Commit message: PCB near end
Parts:
- added R6: 10k, Resistor_THT:R_Axial_DIN0204_L3.6mm_D1.6mm_P7.62mm_Horizontal, F.Cu at (144.0, 88.7)
- added R7: 10k, Resistor_THT:R_Axial_DIN0204_L3.6mm_D1.6mm_P7.62mm_Horizontal, F.Cu at (159.0, 88.7)
- added R8: 10k, Resistor_THT:R_Axial_DIN0204_L3.6mm_D1.6mm_P7.62mm_Horizontal, F.Cu at (174.0, 88.7)
- added R9: 10k, Resistor_THT:R_Axial_DIN0204_L3.6mm_D1.6mm_P7.62mm_Horizontal, F.Cu at (193.0, 88.7)
- added U5: L7805, Package_TO_SOT_THT:TO-220-3_Vertical, F.Cu at (94.4, 36.9)
- moved R5 74.1 mm to (198.0, 25.2)
- moved Q4 73.1 mm to (195.5, 41.5)
- moved R4 69.4 mm to (175.5, 25.2)
- moved Q3 68.4 mm to (173.0, 41.5)
- moved U4 68.3 mm to (198.0, 57.0)
- moved R3 67.2 mm to (156.0, 25.2)
- moved Q2 66.0 mm to (153.5, 41.5)
- moved U3 63.8 mm to (175.5, 57.0)
- moved R2 63.4 mm to (135.0, 25.2)
- moved Q1 62.2 mm to (132.5, 41.5)
- moved U2 60.5 mm to (156.0, 57.0)
- moved D1 59.5 mm to (112.0, 59.0)
- moved R1 57.3 mm to (112.0, 32.2), turned to -90 degrees
- moved U1 56.5 mm to (135.0, 56.9)
- moved J3 54.9 mm to (146.6, 77.0)
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Connections:
- J1 pad 20: Vcc -> Vin_esp
Routing:
- net LEFT1: track 18.8 -> 216.4 mm
- net RIGHT2: track 74.5 -> 260.1 mm
- net LEFT2: track 34.8 -> 167.4 mm
- net RIGHT1: track 169.1 -> 219.9 mm
- net M4: track 42.7 -> 78.2 mm
- net Net-(Q13-Pad2): track 124.5 -> 156.5 mm
- net Gnd: track 0.00 -> 31.9 mm
- net EMERGENCY: track 66.4 -> 94.6 mm
- net M1: track 114.3 -> 86.3 mm
- net M2: track 86.9 -> 66.4 mm
- net M3: track 75.0 -> 57.7 mm
- net Vcc: track 267.1 -> 254.1 mm
- net Net-(Q2-Pad2): track 15.1 -> 24.1 mm
- net Net-(Q1-Pad2): track 15.2 -> 23.7 mm
- net Net-(Q4-Pad2): track 15.1 -> 23.5 mm
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
Commit message: pcb
Parts:
- added J4: Conn_01x05_Male, Connector_PinHeader_2.54mm:PinHeader_1x05_P2.54mm_Vertical, F.Cu at (112.5, 112.0)
- moved J2 2.00 mm to (58.8, 105.0)
Connections:
- J1 pad 10: unconnected-(J1-Pad10) -> PIN1
- J1 pad 6: unconnected-(J1-Pad6) -> PIN5
- J1 pad 7: unconnected-(J1-Pad7) -> PIN4
- J1 pad 8: unconnected-(J1-Pad8) -> PIN3
- J1 pad 9: unconnected-(J1-Pad9) -> PIN2
Routing:
- net PIN4: track 0.00 -> 58.3 mm
- net PIN1: track 0.00 -> 43.7 mm
- net PIN5: track 0.00 -> 42.4 mm
- net PIN2: track 0.00 -> 38.7 mm
- net PIN3: track 0.00 -> 35.4 mm
- net Vin_esp: track 0.00 -> 29.2 mm
- net EMERGENCY: track 94.6 -> 82.6 mm
- added copper zone on B.Cu, net Gnd
- added copper zone on F.Cu, net Gnd
Other:
- board outline added: 171.5 x 113.5 mm
